File: kicad_project/kicad_project.kicad_sch (KiCad schematic)
At the start: 19 parts, among them J1 Screw_Terminal_01x02, J2 Screw_Terminal_01x02, J3 Screw_Terminal_01x02, U3 Opamp_Dual

Commit message: commit
PCB setup
Parts:
- added TP1: TestPoint, TestPoint:TestPoint_Pad_2.0x2.0mm, symbol Connector:TestPoint
Connections:
- net at C2.1, R4.1, R6.2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: now also TP1.1
Other:
- note added: "ERC work"
- note added: "Power input"
- moved on the sheet: C3, C4, J1, J2, J3, U3C
