File: kicad_project/kicad_project.kicad_sch (KiCad schematic)
At the start: 20 parts, among them J1 Screw_Terminal_01x02, J2 Screw_Terminal_01x02, J3 Screw_Terminal_01x02, U3 Opamp_Dual

Commit message: commit
Parts:
- J1, J2, J3: footprint Connector_PinHeader_1.27mm:PinHeader_1x02_P1.27mm_Horizontal -> Connector_PinHeader_1.27mm:PinHeader_1x02_P1.27mm_Vertical
Other:
- moved on the sheet: C3, C4, J2, U3C
